Commit message: initial commit after fork

File: rotors_description/urdf/ardrone.xacro (robot description, xacro)
@@ -20,5 +20,6 @@
   <xacro:property name="sin30" value="0.5" />
   <xacro:property name="cos30" value="0.866025403784" />
-  <xacro:property name="sqrt2" value="1.4142135623730951" />
+  <!-- <xacro:property name="sqrt2" value="1.4142135623730951" /> -->
+  <xacro:property name="sqrt2" value="0.707" />
   <xacro:property name="rotor_drag_coefficient" value="8.06428e-05" />
   <xacro:property name="rolling_moment_coefficient" value="0.000001" />

File: rotors_description/urdf/crazyflie2.xacro (robot description, xacro)
@@ -18,9 +18,9 @@
   <!-- Properties (Taken from Novel Dynamic Inversion Architecture Design for Quadrocopter Control by Jian Wang et al.) -->
   <xacro:property name="namespace" value="$(arg mav_name)" />
-  <xacro:property name="rotor_velocity_slowdown_sim" value="50" />
+  <xacro:property name="rotor_velocity_slowdown_sim" value="10" />
   <xacro:property name="use_mesh_file" value="true" />
   <xacro:property name="mesh_file" value="package://rotors_description/meshes/crazyflie2.dae" />
   <xacro:property name="mass" value="0.025" /> <!-- [kg] -->
-  <xacro:property name="body_width" value="0.045" /> <!-- [m] -->
+  <xacro:property name="body_width" value="0.035" /> <!-- [m] -->
   <xacro:property name="body_height" value="0.03" /> <!-- [m] -->
   <xacro:property name="mass_rotor" value="0.0005" /> <!-- [kg] -->
@@ -35,10 +35,12 @@
   <xacro:property name="time_constant_up" value="0.0125" /> <!-- [s] -->
   <xacro:property name="time_constant_down" value="0.025" /> <!-- [s] -->
-  <xacro:property name="max_rot_velocity" value="2618" /> <!-- [rad/s] -->
+  <xacro:property name="max_rot_velocity" value="5000" /> <!-- 2618[rad/s] -->
   <xacro:property name="rotor_drag_coefficient" value="8.06428e-05" />
+  <!-- <xacro:property name="rotor_drag_coefficient" value="1.8580e-05" /> -->
   <xacro:property name="rolling_moment_coefficient" value="0.000001" />
   <!-- Property Blocks -->
   <xacro:property name="body_inertia">
     <inertia ixx="1.657171e-05" ixy="0.0" ixz="0.0" iyy="1.657171e-05" iyz="0.0" izz="2.9261652e-05" />
+    <!-- <inertia ixx="2.3951e-5" ixy="0.0" ixz="0.0" iyy="2.3951e-5" iyz="0.0" izz="3.2347e-5" /> -->
   </xacro:property>
   <!-- inertia of a single rotor, assuming it is a cuboid. Height=0.4mm, width=0.8mm -->
